Commit message: Correct xacro bugs

File: urdf/human_arm.urdf.xacro (robot description, xacro)
@@ -2,5 +2,5 @@
 <robot xmlns:xacro="http://playerstage.sourceforge.net/gazebo/xmlschema/#interface" name="human_model" >
 <xacro:include filename="props_global.urdf.xacro" />
-<xacro:macro name="human_arm" params="side reflect">
+<xacro:macro name="human_arm" params="side reflect boolside">
     <link name="${side}_arm_mount"/>
     <link name="${side}_shoulder_0"/>
@@ -46,11 +46,22 @@
           <limit lower="${-PI_DIV_2}" upper="${PI_DIV_2}" effort="${max_effort}" velocity="${max_velocity}"  />
         </joint>
-        <joint name="${side}_shoulder_1" type="revolute">
-          <origin xyz="0 0 0" rpy="0 0 0" />
-          <axis xyz="0 0 1" />
-          <parent link="${side}_shoulder_0" />
-          <child link="${side}_shoulder_1" />
-          <limit lower="${-reflect*3PI_DIV_4}" upper="${reflect*PI_DIV_2}" effort="${max_effort}" velocity="${max_velocity}"  />
-        </joint>
+        <xacro:if value="${boolside}">
+          <joint name="right_shoulder_1" type="revolute">
+            <origin xyz="0 0 0" rpy="0 0 0" />
+            <axis xyz="0 0 1" />
+            <parent link="right_shoulder_0" />
+            <child link="right_shoulder_1" />
+            <limit lower="${-PI_DIV_2}" upper="${TPI_DIV_4}" effort="${max_effort}" velocity="${max_velocity}"  />
+          </joint>
+        </xacro:if>
+        <xacro:unless value="${boolside}">
+          <joint name="left_shoulder_1" type="revolute">
+            <origin xyz="0 0 0" rpy="0 0 0" />
+            <axis xyz="0 0 1" />
+            <parent link="left_shoulder_0" />
+            <child link="left_shoulder_1" />
+            <limit lower="${-TPI_DIV_4}" upper="${PI_DIV_2}" effort="${max_effort}" velocity="${max_velocity}"  />
+          </joint>
+        </xacro:unless>
         <joint name="${side}_shoulder_2" type="revolute">
           <origin xyz="0 0 0" rpy="0 0 0" />
@@ -61,11 +72,22 @@
         </joint>
     <!-- END SHOULDER -->
-    <joint name="${side}_elbow_0" type="revolute">
-      <origin xyz="${upper_arm_length} 0 0" rpy="0 0 0" />
-      <axis xyz="0 0 1" />
-      <parent link="${side}_upper_arm" />
-      <child link="${side}_elbow_0" />
-      <limit lower="0.0" upper="${-reflect*PI}" effort="${max_effort}" velocity="${max_velocity}"  />
-    </joint>
+    <xacro:if value="${boolside}">
+      <joint name="right_elbow_0" type="revolute">
+        <origin xyz="${upper_arm_length} 0 0" rpy="0 0 0" />
+        <axis xyz="0 0 1" />
+        <parent link="right_upper_arm" />
+        <child link="right_elbow_0" />
+        <limit lower="0.0" upper="${PI}" effort="${max_effort}" velocity="${max_velocity}"  />
+      </joint>
+    </xacro:if>
+    <xacro:unless value="${boolside}">
+      <joint name="left_elbow_0" type="revolute">
+        <origin xyz="${upper_arm_length} 0 0" rpy="0 0 0" />
+        <axis xyz="0 0 1" />
+        <parent link="left_upper_arm" />
+        <child link="left_elbow_0" />
+        <limit lower="${-PI}" upper="0.0" effort="${max_effort}" velocity="${max_velocity}"  />
+      </joint>
+    </xacro:unless>
     <joint name="${side}_elbow_1" type="revolute">
       <origin xyz="0 0 0" rpy="0 0 0" />
@@ -73,5 +95,5 @@
       <parent link="${side}_elbow_0" />
       <child link="${side}_forearm" />
-      <limit lower="0.0" upper="${-reflect*PI}" effort="${max_effort}" velocity="${max_velocity}"  />
+      <limit lower="${-PI}" upper="${PI}" effort="${max_effort}" velocity="${max_velocity}"  />
     </joint>
     <!-- WRIST : spherical -->

File: urdf/human_skeleton.urdf.xacro (robot description, xacro)
@@ -6,6 +6,6 @@
    <xacro:include filename="props_global.urdf.xacro" />
    <xacro:human_body />
-   <xacro:human_arm side="right" reflect="-1"/>
-   <xacro:human_arm side="left" reflect="1"/>
+   <xacro:human_arm side="right" reflect="-1" boolside="0"/>
+   <xacro:human_arm side="left" reflect="1" boolside="1"/>
    <xacro:human_leg side="right" reflect="-1"/>
    <xacro:human_leg side="left" reflect="1"/>

File: urdf/people/human.urdf (robot description, URDF)
Before this commit: robot human_model, 38 links, 37 joints
Links:
- link left_forearm: geometry visual cylinder length=0.205104157797 radius=0.025
- link left_shin: geometry visual cylinder length=0.470162466925 radius=0.025
- link left_thigh: geometry visual cylinder length=0.507560229301 radius=0.05
- link left_upper_arm: geometry visual cylinder length=0.271329836892 radius=0.05
- link right_forearm: geometry visual cylinder length=0.205104157797 radius=0.025
- link right_shin: geometry visual cylinder length=0.470162466925 radius=0.025
- link right_thigh: geometry visual cylinder length=0.507560229301 radius=0.05
- link right_upper_arm: geometry visual cylinder length=0.271329836892 radius=0.05
- link torso: geometry visual cylinder length=0.312779626643 radius=0.15
- link waist: geometry visual cylinder length=0.0732617665986 radius=0.12
Joints:
- joint left_ankle_0: origin xyz=0.326688842114 0 0 rpy=-1.57079632679 0 1.57079632679 -> xyz=0.470162466925 0 0 rpy=-1.57079632679 0 1.57079632679
- joint left_arm_mount: origin xyz=0 0.195550085817 0.274845351562 rpy=0 0 1.57079632679 -> xyz=0 0.195284400097 0.210067904481 rpy=0 0 1.57079632679
- joint left_elbow_0: limit lower=0.0 upper=-3.14159265359 effort=1 velocity=1 -> lower=-3.14159265359 upper=0.0 effort=1 velocity=1; origin xyz=0.259726985647 0 0 rpy=0 0 0 -> xyz=0.271329836892 0 0 rpy=0 0 0
- joint left_elbow_1: limit lower=0.0 upper=-3.14159265359 effort=1 velocity=1 -> lower=-3.14159265359 upper=3.14159265359 effort=1 velocity=1
- joint left_hip_leg_mount: origin xyz=0 0.0833368553699 -0.0855006138046 rpy=0 1.57079632679 0 -> xyz=0 0.0661475518415 -0.0946929458205 rpy=0 1.57079632679 0
- joint left_knee: origin xyz=0.60022618697 0 0 rpy=1.57079632679 0 0 -> xyz=0.507560229301 0 0 rpy=1.57079632679 0 0
- joint left_shoulder_1: limit lower=-3.0 upper=1.57079632679 effort=1 velocity=1 -> lower=-2.35619449019 upper=1.57079632679 effort=1 velocity=1
- joint left_wrist_0: origin xyz=0.216225022397 0 0 rpy=0 0 0 -> xyz=0.205104157797 0 0 rpy=0 0 0
- joint neck_0: origin xyz=0 0 0.376309040407 rpy=0 0 0 -> xyz=0 0 0.312779626643 rpy=0 0 0
- joint right_ankle_0: origin xyz=0.326688842114 0 0 rpy=-1.57079632679 0 1.57079632679 -> xyz=0.470162466925 0 0 rpy=-1.57079632679 0 1.57079632679
- joint right_arm_mount: origin xyz=0 -0.195550085817 0.274845351562 rpy=0 0 -1.57079632679 -> xyz=0 -0.195284400097 0.210067904481 rpy=0 0 -1.57079632679
- joint right_elbow_0: origin xyz=0.259726985647 0 0 rpy=0 0 0 -> xyz=0.271329836892 0 0 rpy=0 0 0
- joint right_elbow_1: limit lower=0.0 upper=3.14159265359 effort=1 velocity=1 -> lower=-3.14159265359 upper=3.14159265359 effort=1 velocity=1
- joint right_hip_leg_mount: origin xyz=0 -0.0833368553699 -0.0855006138046 rpy=0 1.57079632679 0 -> xyz=0 -0.0661475518415 -0.0946929458205 rpy=0 1.57079632679 0
- joint right_knee: origin xyz=0.60022618697 0 0 rpy=1.57079632679 0 0 -> xyz=0.507560229301 0 0 rpy=1.57079632679 0 0
- joint right_shoulder_1: limit lower=3.0 upper=-1.57079632679 effort=1 velocity=1 -> lower=-1.57079632679 upper=2.35619449019 effort=1 velocity=1
- joint right_wrist_0: origin xyz=0.216225022397 0 0 rpy=0 0 0 -> xyz=0.205104157797 0 0 rpy=0 0 0
- joint spine_0: origin xyz=0 0 0.0874953789355 rpy=0 0 0 -> xyz=0 0 0.0732617665986 rpy=0 0 0

File: urdf/props_global.urdf.xacro (robot description, xacro)
@@ -3,5 +3,5 @@
   <xacro:property name="PI" value="3.14159265359" />
   <xacro:property name="PI_DIV_2" value="1.5707963267948966" />
-  <xacro:property name="3PI_DIV_4" value="2.35619449019" />
+  <xacro:property name="TPI_DIV_4" value="2.35619449019" />
   <xacro:property name="insignificant_mass" value="0.0001" />
   <xacro:property name="insig_inert_xx" value="0.00000001" />

Commit message: Correct URDF
- Add end-effectors joints
- Correct side errors on arms

File: urdf/human_arm.urdf.xacro (robot description, xacro)
@@ -32,4 +32,5 @@
       </visual>
     </link>
+    <link name="${side}_hand_tip"/>
     <!-- Joints -->
     <joint name="${side}_arm_mount" type="fixed">
@@ -47,4 +48,13 @@
         </joint>
         <xacro:if value="${boolside}">
+          <joint name="left_shoulder_1" type="revolute">
+            <origin xyz="0 0 0" rpy="0 0 0" />
+            <axis xyz="0 0 1" />
+            <parent link="left_shoulder_0" />
+            <child link="left_shoulder_1" />
+            <limit lower="${-TPI_DIV_4}" upper="${PI_DIV_2}" effort="${max_effort}" velocity="${max_velocity}"  />
+          </joint>
+        </xacro:if>
+        <xacro:unless value="${boolside}">
           <joint name="right_shoulder_1" type="revolute">
             <origin xyz="0 0 0" rpy="0 0 0" />
@@ -53,13 +63,4 @@
             <child link="right_shoulder_1" />
             <limit lower="${-PI_DIV_2}" upper="${TPI_DIV_4}" effort="${max_effort}" velocity="${max_velocity}"  />
-          </joint>
-        </xacro:if>
-        <xacro:unless value="${boolside}">
-          <joint name="left_shoulder_1" type="revolute">
-            <origin xyz="0 0 0" rpy="0 0 0" />
-            <axis xyz="0 0 1" />
-            <parent link="left_shoulder_0" />
-            <child link="left_shoulder_1" />
-            <limit lower="${-TPI_DIV_4}" upper="${PI_DIV_2}" effort="${max_effort}" velocity="${max_velocity}"  />
           </joint>
         </xacro:unless>
@@ -73,4 +74,13 @@
     <!-- END SHOULDER -->
     <xacro:if value="${boolside}">
+      <joint name="left_elbow_0" type="revolute">
+        <origin xyz="${upper_arm_length} 0 0" rpy="0 0 0" />
+        <axis xyz="0 0 1" />
+        <parent link="left_upper_arm" />
+        <child link="left_elbow_0" />
+        <limit lower="${-PI}" upper="0.1" effort="${max_effort}" velocity="${max_velocity}"  />
+      </joint>
+    </xacro:if>
+    <xacro:unless value="${boolside}">
       <joint name="right_elbow_0" type="revolute">
         <origin xyz="${upper_arm_length} 0 0" rpy="0 0 0" />
@@ -78,14 +88,5 @@
         <parent link="right_upper_arm" />
         <child link="right_elbow_0" />
-        <limit lower="0.0" upper="${PI}" effort="${max_effort}" velocity="${max_velocity}"  />
-      </joint>
-    </xacro:if>
-    <xacro:unless value="${boolside}">
-      <joint name="left_elbow_0" type="revolute">
-        <origin xyz="${upper_arm_length} 0 0" rpy="0 0 0" />
-        <axis xyz="0 0 1" />
-        <parent link="left_upper_arm" />
-        <child link="left_elbow_0" />
-        <limit lower="${-PI}" upper="0.0" effort="${max_effort}" velocity="${max_velocity}"  />
+        <limit lower="-0.1" upper="${PI}" effort="${max_effort}" velocity="${max_velocity}"  />
       </joint>
     </xacro:unless>
@@ -113,4 +114,9 @@
         </joint>
     <!-- END WRIST -->
+    <joint name="${side}_hand" type="fixed">
+      <origin xyz="${hand_length} 0 0" rpy="0 0 0" />
+      <parent link="${side}_hand" />
+      <child link="${side}_hand_tip" />
+    </joint>
 </xacro:macro>
 </robot>

File: urdf/human_body.urdf.xacro (robot description, xacro)
@@ -34,4 +34,5 @@
       </visual>
     </link>
+    <link name="head_tip"/>
     <joint name="hip" type="fixed">
       <origin xyz="0 0 0" rpy="0 0 0" />
@@ -84,4 +85,9 @@
         </joint>
     <!-- END NECK -->
+    <joint name="head" type="fixed">
+      <origin xyz="0 0 ${neck_length}" rpy="0 0 0" />
+      <parent link="head" />
+      <child link="head_tip" />
+    </joint>
 </xacro:macro>
 </robot>

File: urdf/human_leg.urdf.xacro (robot description, xacro)
@@ -31,4 +31,5 @@
       </visual>
     </link>
+    <link name="${side}_foot_tip"/>
     <!-- Joints -->
     <joint name="${side}_hip_leg_mount" type="fixed">
@@ -65,5 +66,5 @@
       <parent link="${side}_thigh" />
       <child link="${side}_shin" />
-      <limit lower="${-PI}" upper="0" effort="${max_effort}" velocity="${max_velocity}"  />
+      <limit lower="${-PI}" upper="0.1" effort="${max_effort}" velocity="${max_velocity}"  />
     </joint>
     <!-- ankle : spherical -->
@@ -83,4 +84,9 @@
         </joint>
     <!-- END ankle -->
+    <joint name="${side}_foot" type="fixed">
+      <origin xyz="${foot_length} 0 0" rpy="0 0 0" />
+      <parent link="${side}_foot" />
+      <child link="${side}_foot_tip" />
+    </joint>
 </xacro:macro>
 </robot>

File: urdf/people/human.urdf (robot description, URDF)
Before this commit: robot human_model, 38 links, 37 joints
Links:
- added link head_tip
- added link left_foot_tip
- added link left_hand_tip
- added link right_foot_tip
- added link right_hand_tip
- link left_forearm: geometry visual cylinder length=0.263379948718 radius=0.025
- link left_shin: geometry visual cylinder length=0.313345772978 radius=0.025
- link left_thigh: geometry visual cylinder length=0.443948434173 radius=0.05
- link left_upper_arm: geometry visual cylinder length=0.242967916466 radius=0.05
- link right_forearm: geometry visual cylinder length=0.263379948718 radius=0.025
- link right_shin: geometry visual cylinder length=0.313345772978 radius=0.025
- link right_thigh: geometry visual cylinder length=0.443948434173 radius=0.05
- link right_upper_arm: geometry visual cylinder length=0.242967916466 radius=0.05
- link torso: geometry visual cylinder length=0.31994599126 radius=0.15
- link waist: geometry visual cylinder length=0.0756640482208 radius=0.12
Joints:
- added joint head: type fixed, parent head, child head_tip, origin xyz=0 0 0.182430717129 rpy=0 0 0
- added joint left_foot: type fixed, parent left_foot, child left_foot_tip, origin xyz=0.1 0 0 rpy=0 0 0
- added joint left_hand: type fixed, parent left_hand, child left_hand_tip, origin xyz=0.1 0 0 rpy=0 0 0
- added joint right_foot: type fixed, parent right_foot, child right_foot_tip, origin xyz=0.1 0 0 rpy=0 0 0
- added joint right_hand: type fixed, parent right_hand, child right_hand_tip, origin xyz=0.1 0 0 rpy=0 0 0
- joint left_ankle_0: origin xyz=0.470162466925 0 0 rpy=-1.57079632679 0 1.57079632679 -> xyz=0.313345772978 0 0 rpy=-1.57079632679 0 1.57079632679
- joint left_arm_mount: origin xyz=0 0.195284400097 0.210067904481 rpy=0 0 1.57079632679 -> xyz=0 0.191025299573 0.230898322182 rpy=0 0 1.57079632679
- joint left_elbow_0: limit lower=-3.14159265359 upper=0.0 effort=1 velocity=1 -> lower=-3.14159265359 upper=0.1 effort=1 velocity=1; origin xyz=0.271329836892 0 0 rpy=0 0 0 -> xyz=0.242967916466 0 0 rpy=0 0 0
- joint left_hip_leg_mount: origin xyz=0 0.0661475518415 -0.0946929458205 rpy=0 1.57079632679 0 -> xyz=0 0.0764992904338 -0.0838923317292 rpy=0 1.57079632679 0
- joint left_knee: origin xyz=0.507560229301 0 0 rpy=1.57079632679 0 0 -> xyz=0.443948434173 0 0 rpy=1.57079632679 0 0
- joint left_wrist_0: origin xyz=0.205104157797 0 0 rpy=0 0 0 -> xyz=0.263379948718 0 0 rpy=0 0 0
- joint neck_0: origin xyz=0 0 0.312779626643 rpy=0 0 0 -> xyz=0 0 0.31994599126 rpy=0 0 0
- joint right_ankle_0: origin xyz=0.470162466925 0 0 rpy=-1.57079632679 0 1.57079632679 -> xyz=0.313345772978 0 0 rpy=-1.57079632679 0 1.57079632679
- joint right_arm_mount: origin xyz=0 -0.195284400097 0.210067904481 rpy=0 0 -1.57079632679 -> xyz=0 -0.191025299573 0.230898322182 rpy=0 0 -1.57079632679
- joint right_elbow_0: limit lower=0.0 upper=3.14159265359 effort=1 velocity=1 -> lower=-0.1 upper=3.14159265359 effort=1 velocity=1; origin xyz=0.271329836892 0 0 rpy=0 0 0 -> xyz=0.242967916466 0 0 rpy=0 0 0
- joint right_hip_leg_mount: origin xyz=0 -0.0661475518415 -0.0946929458205 rpy=0 1.57079632679 0 -> xyz=0 -0.0764992904338 -0.0838923317292 rpy=0 1.57079632679 0
- joint right_knee: origin xyz=0.507560229301 0 0 rpy=1.57079632679 0 0 -> xyz=0.443948434173 0 0 rpy=1.57079632679 0 0
- joint right_wrist_0: origin xyz=0.205104157797 0 0 rpy=0 0 0 -> xyz=0.263379948718 0 0 rpy=0 0 0
- joint spine_0: origin xyz=0 0 0.0732617665986 rpy=0 0 0 -> xyz=0 0 0.0756640482208 rpy=0 0 0

Commit message: Change URDF for better joint limits

File: urdf/human_arm.urdf.xacro (robot description, xacro)
@@ -79,5 +79,12 @@
         <parent link="left_upper_arm" />
         <child link="left_elbow_0" />
-        <limit lower="${-PI}" upper="0.1" effort="${max_effort}" velocity="${max_velocity}"  />
+        <limit lower="${-PI}" upper="0.0" effort="${max_effort}" velocity="${max_velocity}"  />
+      </joint>
+      <joint name="left_elbow_1" type="revolute">
+        <origin xyz="0 0 0" rpy="0 0 0" />
+        <axis xyz="1 0 0" />
+        <parent link="left_elbow_0" />
+        <child link="left_forearm" />
+        <limit lower="${-PI}" upper="0.0" effort="${max_effort}" velocity="${max_velocity}"  />
       </joint>
     </xacro:if>
@@ -88,30 +95,28 @@
         <parent link="right_upper_arm" />
         <child link="right_elbow_0" />
-        <limit lower="-0.1" upper="${PI}" effort="${max_effort}" velocity="${max_velocity}"  />
+        <limit lower="0.0" upper="${PI}" effort="${max_effort}" velocity="${max_velocity}"  />
+      </joint>
+      <joint name="right_elbow_1" type="revolute">
+        <origin xyz="0 0 0" rpy="0 0 0" />
+        <axis xyz="1 0 0" />
+        <parent link="right_elbow_0" />
+        <child link="right_forearm" />
+        <limit lower="0.0" upper="${PI}" effort="${max_effort}" velocity="${max_velocity}"  />
       </joint>
     </xacro:unless>
-    <joint name="${side}_elbow_1" type="revolute">
+    <joint name="${side}_wrist_0" type="revolute">
+      <origin xyz="${forearm_length} 0 0" rpy="0 0 0" />
+      <axis xyz="0 0 1" />
+      <parent link="${side}_forearm" />
+      <child link="${side}_wrist_0" />
+      <limit lower="${-PI_DIV_4}" upper="${PI_DIV_4}" effort="${max_effort}" velocity="${max_velocity}"  />
+    </joint>
+    <joint name="${side}_wrist_1" type="revolute">
       <origin xyz="0 0 0" rpy="0 0 0" />
-      <axis xyz="1 0 0" />
-      <parent link="${side}_elbow_0" />
-      <child link="${side}_forearm" />
-      <limit lower="${-PI}" upper="${PI}" effort="${max_effort}" velocity="${max_velocity}"  />
+      <axis xyz="0 1 0" />
+      <parent link="${side}_wrist_0" />
+      <child link="${side}_hand" />
+      <limit lower="${-PI_DIV_2}" upper="${PI_DIV_2}" effort="${max_effort}" velocity="${max_velocity}"  />
     </joint>
-    <!-- WRIST : spherical -->
-        <joint name="${side}_wrist_0" type="revolute">
-          <origin xyz="${forearm_length} 0 0" rpy="0 0 0" />
-          <axis xyz="0 0 1" />
-          <parent link="${side}_forearm" />
-          <child link="${side}_wrist_0" />
-          <limit lower="${-PI_DIV_2}" upper="${PI_DIV_2}" effort="${max_effort}" velocity="${max_velocity}"  />
-        </joint>
-        <joint name="${side}_wrist_1" type="revolute">
-          <origin xyz="0 0 0" rpy="0 0 0" />
-          <axis xyz="0 1 0" />
-          <parent link="${side}_wrist_0" />
-          <child link="${side}_hand" />
-          <limit lower="${-PI_DIV_2}" upper="${PI_DIV_2}" effort="${max_effort}" velocity="${max_velocity}"  />
-        </joint>
-    <!-- END WRIST -->
     <joint name="${side}_hand" type="fixed">
       <origin xyz="${hand_length} 0 0" rpy="0 0 0" />

File: urdf/props_global.urdf.xacro (robot description, xacro)
@@ -3,4 +3,5 @@
   <xacro:property name="PI" value="3.14159265359" />
   <xacro:property name="PI_DIV_2" value="1.5707963267948966" />
+  <xacro:property name="PI_DIV_4" value="0.78539816339" />
   <xacro:property name="TPI_DIV_4" value="2.35619449019" />
   <xacro:property name="insignificant_mass" value="0.0001" />
